Commit message: 物料的抓取与放置仿真

File: 11projects/07pick_place/src/common_pkg/urdf/material.urdf.xacro (robot description, xacro)
@@ -4,5 +4,5 @@
     <xacro:property name="box_y" value="0.06" />
     <xacro:property name="box_z" value="0.16" />
-    <xacro:property name="box_mass" value="0.05" />
+    <xacro:property name="box_mass" value="0.5" />
     <link name="material_link">
         <inertial>
@@ -18,5 +18,5 @@
             <origin xyz="0 0 ${box_z/2}" />
             <geometry>
-                <box size="0.06 0.06 0.16" />
+                <box size="${box_x} ${box_y} ${box_z}" />
             </geometry>
         </visual>
@@ -32,4 +32,6 @@
         <mu1>1.0</mu1>
         <mu2>1.0</mu2>
+        <kp>1000000.0</kp>
+        <kd>1.0</kd>
     </gazebo>
 </robot>

File: 11projects/07pick_place/src/robot_description/urdf/robot.urdf.xacro (robot description, xacro)
@@ -14,5 +14,5 @@
         <parent link="stage_slide_link" />
         <child link="base_link"/>
-        <origin rpy="-${pi/2} 0 0" />
+        <origin rpy="${pi/2} 0 0" />
     </joint>
     <!-- load arm  -->

File: 11projects/07pick_place/src/stage_description/urdf/stage.urdf.xacro (robot description, xacro)
@@ -46,5 +46,5 @@
     <link name="stage_slide_link" >
       <visual>
-         <origin xyz="0 ${slide_y/2} 0" />
+         <origin xyz="0 -${slide_y/2} 0" />
           <geometry>
               <box size="${slide_x} ${slide_y} ${slide_z}"/>
@@ -55,5 +55,5 @@
       </visual>
       <collision>
-         <origin xyz="0 ${slide_y/2} 0" />
+         <origin xyz="0 -${slide_y/2} 0" />
           <geometry>
               <box size="${slide_x} ${slide_y} ${slide_z}"/>
@@ -64,5 +64,5 @@
       </collision>
       <xacro:box_inertial x="${slide_x}" y="${slide_y}" z="${slide_z}" mass="${slide_mass}">
-         <origin xyz="0 ${slide_y/2} 0" />
+         <origin xyz="0 -${slide_y/2} 0" />
       </xacro:box_inertial>
     </link>
@@ -70,5 +70,5 @@
       <parent link="stage_base_link" />
       <child link = "stage_slide_link" />
-      <origin xyz="0 0 ${stage_z}" rpy="${pi/2} 0 0" />
+      <origin xyz="0 0 ${stage_z}" rpy="-${pi/2} 0 0" />
       <axis xyz="0 0 1" />
       <limit lower="-${(stage_y - slide_z)/2}" upper="${(stage_y - slide_z)/2}" effort="400" velocity="1"/>

Commit message: 物料的抓取与放置仿真

File: 11projects/07pick_place/src/common_pkg/urdf/material.urdf.xacro (robot description, xacro)
@@ -4,5 +4,5 @@
     <xacro:property name="box_y" value="0.06" />
     <xacro:property name="box_z" value="0.16" />
-    <xacro:property name="box_mass" value="0.5" />
+    <xacro:property name="box_mass" value="0.8" />
     <link name="material_link">
         <inertial>

File: 11projects/07pick_place/src/robot_description/urdf/common.gazebo.xacro (robot description, xacro)
@@ -8,3 +8,24 @@
          </plugin>
      </gazebo>
+    <gazebo>
+    <!-- you need install from https://github.com/JenniferBuehler/gazebo-pkgs/tree/master/gazebo_grasp_plugin
+    and place the .so file to $GAZEBO_PLUGIN_PATH,default path is /usr/lib/x86_64-linux-gnu/gazebo-9/plugins
+    -->
+        <plugin name="gazebo_grasp_fix" filename="libgazebo_grasp_fix.so">
+            <arm>
+                <arm_name>arm</arm_name>
+                <palm_link>Link1</palm_link>
+                <gripper_link>Link11</gripper_link>
+                <palm_link>Link2</palm_link>
+                <gripper_link>Link22</gripper_link>
+            </arm>
+            <forces_angle_tolerance>100</forces_angle_tolerance>
+            <update_rate>20</update_rate>
+            <grip_count_threshold>1</grip_count_threshold>
+            <max_grip_count>3</max_grip_count>
+            <release_tolerance>0.0198</release_tolerance>
+            <disable_collisions_on_attach>false</disable_collisions_on_attach>
+            <contact_topic>__default_topic__</contact_topic>
+        </plugin>
+    </gazebo>
 </robot>
